File: arduino_uno.kicad_sch (KiCad schematic)
At the start: 4 parts, among them J1 Power, J2 Digital/PWM, J3 Analog, J4 Digital/PWM

Commit message: fix erc
Connections:
- net *10: no longer names the net of J2.8 (Pin_8)
- net *11: no longer names the net of J2.7 (Pin_7)
- net *3: no longer names the net of J4.5 (Pin_5)
- net *5: no longer names the net of J4.3 (Pin_3)
- net *6: no longer names the net of J4.2 (Pin_2)
- net *9: no longer names the net of J2.9 (Pin_9)
- net 12: no longer names the net of J2.6 (Pin_6)
- net 13: no longer names the net of J2.5 (Pin_5)
- net 2: no longer names the net of J4.6 (Pin_6)
- net 4: no longer names the net of J4.4 (Pin_4)
- net 7: no longer names the net of J4.1 (Pin_1)
- net 8: no longer names the net of J2.10 (Pin_10)
- net A0: no longer names the net of J3.1 (Pin_1)
- net A1: no longer names the net of J3.2 (Pin_2)
- net A2: no longer names the net of J3.3 (Pin_3)
- net A3: no longer names the net of J3.4 (Pin_4)
- net AREF: no longer names the net of J2.3 (Pin_3)
- net IOREF: no longer names the net of J1.2 (Pin_2)
- net RX/0: no longer names the net of J4.8 (Pin_8)
- net TX/1: no longer names the net of J4.7 (Pin_7)
- net ~{RESET}: no longer names the net of J1.3 (Pin_3)
