File: arduino_uno.kicad_pcb (KiCad board)
At the start: 2 copper layers, 68.6 x 53.3 mm, 8 parts, among them J1 Power, J2 Digital/PWM, J3 Analog, J4 Digital/PWM

Commit message: fix drc
Connections:
- J1 pad 2: /IOREF -> unconnected-(J1-Pad2)
- J1 pad 3: /~{RESET} -> unconnected-(J1-Pad3)
- J2 pad 10: /8 -> unconnected-(J2-Pad10)
- J2 pad 3: /AREF -> unconnected-(J2-Pad3)
- J2 pad 5: /13 -> unconnected-(J2-Pad5)
- J2 pad 6: /12 -> unconnected-(J2-Pad6)
- J2 pad 7: /*11 -> unconnected-(J2-Pad7)
- J2 pad 8: /*10 -> unconnected-(J2-Pad8)
- J2 pad 9: /*9 -> unconnected-(J2-Pad9)
- J3 pad 1: /A0 -> unconnected-(J3-Pad1)
- J3 pad 2: /A1 -> unconnected-(J3-Pad2)
- J3 pad 3: /A2 -> unconnected-(J3-Pad3)
- J3 pad 4: /A3 -> unconnected-(J3-Pad4)
- J4 pad 1: /7 -> unconnected-(J4-Pad1)
- J4 pad 2: /*6 -> unconnected-(J4-Pad2)
- J4 pad 3: /*5 -> unconnected-(J4-Pad3)
- J4 pad 4: /4 -> unconnected-(J4-Pad4)
- J4 pad 5: /*3 -> unconnected-(J4-Pad5)
- J4 pad 6: /2 -> unconnected-(J4-Pad6)
- J4 pad 7: /TX/1 -> unconnected-(J4-Pad7)
- J4 pad 8: /RX/0 -> unconnected-(J4-Pad8)
Routing:
- net /SCL/A5: track 0.00 -> 66.8 mm
- net /SDA/A4: track 0.00 -> 64.7 mm, vias 0 -> 1
- net GND: track 0.00 -> 56.7 mm
